Commit message: edited paths

File: src/my_robot/description/chassis.urdf.xacro (robot description, xacro)
@@ -1,4 +1,4 @@
 <?xml version="1.0" ?>
-<robot xmlns:xacro="http://ros.org/wiki/xacro" name="chassis.urdf">
+<robot xmlns:xacro="http://www.ros.org/wiki/xacro" name="chassis">
   <xacro:macro name="chassis" params="">
     <link name="baselink">
@@ -14,13 +14,11 @@
         </geometry>
         <material name="white">
-        <color rgba="1 1 1 1"/>
-      </material>
+          <color rgba="1 1 1 1"/>
+        </material>
       </visual>
       <collision>
         <origin rpy="0 0 0" xyz="0 0 0"/>
         <geometry>
-          <mesh filename="chassis.obj" scale="1.0 1.0 1.0"/>
-          <!-- you could also specify the collision (for the chassis) with a "box" tag: -->
-          <!-- <box size=".06 .06 .06"/> -->
+          <mesh filename="package://my_robot/description/chassis.obj" scale="1.0 1.0 1.0"/>
         </geometry>
       </collision>

File: src/my_robot/description/robot.urdf.xacro (robot description, xacro)
@@ -1,4 +1,4 @@
 <?xml version="1.0"?>
-<robot xmlns:xacro="http://ros.org/wiki/xacro" name="my_robot">
+<robot xmlns:xacro="http://www.ros.org/wiki/xacro" name="my_robot">
   <!-- include the chassis -->
   <xacro:include filename="chassis.urdf.xacro"/>

Commit message: urdf construction

File: src/my_robot/description/chassis.urdf.xacro (robot description, xacro)
@@ -2,5 +2,5 @@
 <robot xmlns:xacro="http://www.ros.org/wiki/xacro" name="chassis">
   <xacro:macro name="chassis" params="">
-    <link name="baselink">
+    <link name="base_link">
       <inertial>
         <origin rpy="0 0 0" xyz="0 0 0"/>

File: src/my_robot/description/drive_wheel.urdf.xacro (robot description, xacro)
@@ -1,5 +1,6 @@
 <?xml version="1.0" ?>
-<robot name="drive_wheel.urdf">
-  <link name="baselink">
+<robot xmlns:xacro="http://www.ros.org/wiki/xacro" name="drive_wheel.urdf">
+  <xacro:macro name="drive_wheel" params="wheel_name joint_name parent_link xyz_pos">
+  <link name="${wheel_name}">
     <inertial>
       <origin rpy="0 0 0" xyz="0 0 0"/>
@@ -10,5 +11,5 @@
       <origin rpy="0 0 0" xyz="0 0 0"/>
       <geometry>
-        <mesh filename="drive_wheel.obj" scale="1.0 1.0 1.0"/>
+        <mesh filename="package://my_robot/description/drive_wheel.obj" scale="1.0 1.0 1.0"/>
       </geometry>
       <material name="white">
@@ -19,5 +20,5 @@
       <origin rpy="0 0 0" xyz="0 0 0"/>
       <geometry>
-        <mesh filename="drive_wheel.obj" scale="1.0 1.0 1.0"/>
+        <mesh filename="package://my_robot/description/drive_wheel.obj" scale="1.0 1.0 1.0"/>
         <!-- you could also specify the collision (for the drive_wheel) with a "box" tag: -->
         <!-- <box size=".06 .06 .06"/> -->
@@ -25,3 +26,10 @@
     </collision>
   </link>
+    <joint name="${joint_name}" type="continuous">
+      <parent link="${parent_link}"/>
+      <child link="${wheel_name}"/>
+      <origin xyz="${xyz_pos}" rpy="0 0 0"/>
+      <axis xyz="0 1 0"/>
+    </joint>
+  </xacro:macro>
 </robot>

File: src/my_robot/description/robot.urdf.xacro (robot description, xacro)
@@ -3,11 +3,23 @@
   <!-- include the chassis -->
   <xacro:include filename="chassis.urdf.xacro"/>
+  <xacro:include filename="drive_wheel.urdf.xacro"/>
   <xacro:chassis/>
+  <xacro:drive_wheel
+  wheel_name="left_wheel_link"
+  joint_name="left_wheel_joint"
+  parent_link="base_link"
+  xyz_pos="0.078 0.22 -0.2"/>
+<xacro:drive_wheel
+  wheel_name="right_wheel_link"
+  joint_name="right_wheel_joint"
+  parent_link="base_link"
+  xyz_pos="0.078 -0.22 -0.2"/>
+  <!-- <xacro:drive_wheel/> -->
   <!-- define a root base_link -->
-  <link name="base_link"/>
+  <link name="map"/>
   <!-- fixed joint to attach chassis -->
   <joint name="base_to_chassis" type="fixed">
-    <parent link="base_link"/>
-    <child link="baselink"/>
+    <parent link="map"/>
+    <child link="base_link"/>
     <origin xyz="0 0 0" rpy="0 0 0"/>
   </joint>

Commit message: now with minimal gazebo

File: src/my_robot/description/chassis.urdf.xacro (robot description, xacro)
@@ -5,11 +5,12 @@
       <inertial>
         <origin rpy="0 0 0" xyz="0 0 0"/>
-        <mass value="0.0"/>
-        <inertia ixx="0" ixy="0" ixz="0" iyy="0" iyz="0" izz="0"/>
+        <mass value="1.0"/>
+        <inertia ixx="0.01" iyy="0.01" izz="0.01" ixy="0" ixz="0" iyz="0"/>
       </inertial>
       <visual>
         <origin rpy="0 0 0" xyz="0 0 0"/>
         <geometry>
-          <mesh filename="package://my_robot/description/chassis.obj" scale="1.0 1.0 1.0"/>
+          <!-- <mesh filename="package://my_robot/description/chassis.obj" scale="1.0 1.0 1.0"/> -->
+          <mesh filename="file://$(find my_robot)/description/chassis.obj"/>
         </geometry>
         <material name="white">
@@ -20,8 +21,30 @@
         <origin rpy="0 0 0" xyz="0 0 0"/>
         <geometry>
-          <mesh filename="package://my_robot/description/chassis.obj" scale="1.0 1.0 1.0"/>
+          <!-- <mesh filename="package://my_robot/description/chassis.obj" scale="1.0 1.0 1.0"/> -->
+          <mesh filename="file://$(find my_robot)/description/chassis.obj"/>
         </geometry>
       </collision>
     </link>
   </xacro:macro>
+  <!-- <xacro:macro name="chassis" params="">
+    <link name="base_link">
+      <visual>
+        <origin xyz="0 0 0" rpy="0 0 0"/>
+        <geometry>
+          <box size="0.5 0.3 0.1"/>
+        </geometry>
+        <material name="Gazebo/Red"/>
+      </visual>
+      <collision>
+        <origin xyz="0 0 0" rpy="0 0 0"/>
+        <geometry>
+          <box size="0.5 0.3 0.1"/>
+        </geometry>
+      </collision>
+      <inertial>
+        <mass value="1.0"/>
+        <inertia ixx="0.01" ixy="0" ixz="0" iyy="0.01" iyz="0" izz="0.01"/>
+      </inertial>
+    </link>
+  </xacro:macro> -->
 </robot>

File: src/my_robot/description/drive_wheel.urdf.xacro (robot description, xacro)
@@ -5,11 +5,12 @@
     <inertial>
       <origin rpy="0 0 0" xyz="0 0 0"/>
-       <mass value="0.0"/>
-       <inertia ixx="0" ixy="0" ixz="0" iyy="0" iyz="0" izz="0"/>
+       <mass value="0.5"/>
+       <inertia ixx="0.01" iyy="0.01" izz="0.01" ixy="0" ixz="0" iyz="0"/>
     </inertial>
     <visual>
       <origin rpy="0 0 0" xyz="0 0 0"/>
       <geometry>
-        <mesh filename="package://my_robot/description/drive_wheel.obj" scale="1.0 1.0 1.0"/>
+        <!-- <mesh filename="package://my_robot/description/drive_wheel.obj" scale="1.0 1.0 1.0"/> -->
+        <mesh filename="file://$(find my_robot)/description/drive_wheel.obj"/>
       </geometry>
       <material name="white">
@@ -20,7 +21,6 @@
       <origin rpy="0 0 0" xyz="0 0 0"/>
       <geometry>
-        <mesh filename="package://my_robot/description/drive_wheel.obj" scale="1.0 1.0 1.0"/>
-        <!-- you could also specify the collision (for the drive_wheel) with a "box" tag: -->
-        <!-- <box size=".06 .06 .06"/> -->
+        <!-- <mesh filename="package://my_robot/description/drive_wheel.obj" scale="1.0 1.0 1.0"/> -->
+        <mesh filename="file://$(find my_robot)/description/drive_wheel.obj"/>
       </geometry>
     </collision>
