Commit message: update

File: src/my_robot/description/robot.urdf.xacro (robot description, xacro)
@@ -1,4 +1,5 @@
 <?xml version="1.0"?>
 <robot xmlns:xacro="http://www.ros.org/wiki/xacro" name="my_robot">
+<xacro:macro name="robot" params="">
   <!-- include the chassis -->
   <xacro:include filename="chassis.urdf.xacro"/>
@@ -24,3 +25,4 @@
     <origin xyz="0 0 0" rpy="0 0 0"/>
   </joint>
+</xacro:macro>
 </robot>
