Commit message: urdf update
physical working, left controller

File: src/my_robot/description/castor_wheel.urdf.xacro (robot description, xacro)
@@ -1,14 +1,17 @@
 <?xml version="1.0" ?>
-<robot name="castor_wheel.urdf">
-  <link name="baselink">
+<robot xmlns:xacro="http://www.ros.org/wiki/xacro" name="castor_wheel">
+  <xacro:macro name="castor_wheel" params="xyz_pos">
+  <xacro:property name="parent_link" value="base_link"/>
+  <xacro:property name="child_link"  value="castor_wheel"/>
+  <link name="castor_wheel">
     <inertial>
       <origin rpy="0 0 0" xyz="0 0 0"/>
-       <mass value="0.0"/>
-       <inertia ixx="0" ixy="0" ixz="0" iyy="0" iyz="0" izz="0"/>
+       <mass value="1.0"/>
+       <inertia ixx="0.01" ixy="0.01" ixz="0.01" iyy="0.01" iyz="0" izz="0.01"/>
     </inertial>
     <visual>
       <origin rpy="0 0 0" xyz="0 0 0"/>
       <geometry>
-        <mesh filename="castor_wheel.obj" scale="1.0 1.0 1.0"/>
+        <mesh filename="file://$(find my_robot)/description/castor_wheel.obj" scale="1.0 1.0 1.0"/>
       </geometry>
       <material name="white">
@@ -19,5 +22,5 @@
       <origin rpy="0 0 0" xyz="0 0 0"/>
       <geometry>
-        <mesh filename="castor_wheel.obj" scale="1.0 1.0 1.0"/>
+        <mesh filename="file://$(find my_robot)/description/castor_wheel.obj" scale="1.0 1.0 1.0"/>
         <!-- you could also specify the collision (for the castor_wheel) with a "box" tag: -->
         <!-- <box size=".06 .06 .06"/> -->
@@ -25,3 +28,9 @@
     </collision>
   </link>
+  <joint name="castor_wheel_joint" type="fixed">
+    <parent link="${parent_link}"/>
+    <child link="${child_link}"/>
+    <origin xyz="${xyz_pos}" rpy="0 0 0 "/>
+  </joint>
+  </xacro:macro>
 </robot>

File: src/my_robot/description/robot.urdf.xacro (robot description, xacro)
@@ -5,5 +5,8 @@
   <xacro:include filename="chassis.urdf.xacro"/>
   <xacro:include filename="drive_wheel.urdf.xacro"/>
+  <xacro:include filename="castor_wheel.urdf.xacro"/>
+  <xacro:include filename="robot_cover.urdf.xacro"/>
   <xacro:chassis/>
+  <!-- <xacro:drive_wheel/> -->
   <xacro:drive_wheel
   wheel_name="left_wheel_link"
@@ -11,10 +14,15 @@
   parent_link="base_link"
   xyz_pos="0.078 0.22 -0.2"/>
-<xacro:drive_wheel
+  <xacro:drive_wheel
   wheel_name="right_wheel_link"
   joint_name="right_wheel_joint"
   parent_link="base_link"
   xyz_pos="0.078 -0.22 -0.2"/>
-  <!-- <xacro:drive_wheel/> -->
+  <!-- <xacro:castor_wheel/> -->
+  <xacro:castor_wheel
+  xyz_pos="-0.2 0 -0.225"/>
+  <!-- <xacro:robot_cover/> -->
+  <xacro:robot_cover
+  xyz_pos="-0.06 0.0 0.05"/>s
   <!-- define a root base_link -->
   <link name="map"/>

File: src/my_robot/description/robot_cover.urdf.xacro (robot description, xacro)
@@ -1,5 +1,6 @@
 <?xml version="1.0" ?>
-<robot name="robot_cover.urdf">
-  <link name="baselink">
+<robot xmlns:xacro="http://www.ros.org/wiki/xacro" name="robot_cover.urdf">
+<xacro:macro name="robot_cover" params="xyz_pos">
+  <link name="robot_cover">
     <inertial>
       <origin rpy="0 0 0" xyz="0 0 0"/>
@@ -10,5 +11,5 @@
       <origin rpy="0 0 0" xyz="0 0 0"/>
       <geometry>
-        <mesh filename="robot_cover.obj" scale="1.0 1.0 1.0"/>
+        <mesh filename="file://$(find my_robot)/description/robot_cover.obj" scale="1.0 1.0 1.0"/>
       </geometry>
       <material name="white">
@@ -19,5 +20,5 @@
       <origin rpy="0 0 0" xyz="0 0 0"/>
       <geometry>
-        <mesh filename="robot_cover.obj" scale="1.0 1.0 1.0"/>
+        <mesh filename="file://$(find my_robot)/description/robot_cover.obj" scale="1.0 1.0 1.0"/>
         <!-- you could also specify the collision (for the robot_cover) with a "box" tag: -->
         <!-- <box size=".06 .06 .06"/> -->
@@ -25,3 +26,9 @@
     </collision>
   </link>
+  <joint name="robot_cover_joint" type="fixed">
+    <parent link="base_link"/>
+    <child link="robot_cover"/>
+    <origin xyz="${xyz_pos}" rpy="0 0 0 "/>
+  </joint>
+  </xacro:macro>
 </robot>

Commit message: revered urdf and added friction for caster

File: src/my_robot/description/castor_wheel.urdf.xacro (robot description, xacro)
@@ -28,4 +28,21 @@
     </collision>
   </link>
+  <gazebo reference="castor_wheel">
+    <!-- <material>Gazebo/White</material> -->
+    <collision>
+      <surface>
+        <friction>
+          <ode>
+            <mu>0.0</mu>
+            <mu2>0.0</mu2>
+          </ode>
+        </friction>
+        <bounce/>
+        <contact>
+          <ode/>
+        </contact>
+      </surface>
+    </collision>
+  </gazebo>
   <joint name="castor_wheel_joint" type="fixed">
     <parent link="${parent_link}"/>

File: src/my_robot/description/drive_wheel.urdf.xacro (robot description, xacro)
@@ -1,5 +1,5 @@
 <?xml version="1.0" ?>
 <robot xmlns:xacro="http://www.ros.org/wiki/xacro" name="drive_wheel.urdf">
-  <xacro:macro name="drive_wheel" params="wheel_name joint_name parent_link xyz_pos">
+  <xacro:macro name="drive_wheel" params="wheel_name joint_name parent_link xyz_pos wheel_flipping">
   <link name="${wheel_name}">
     <inertial>
@@ -9,5 +9,5 @@
     </inertial>
     <visual>
-      <origin rpy="0 0 0" xyz="0 0 0"/>
+      <origin rpy="0 0 ${wheel_flipping}" xyz="0 0 0"/>
       <geometry>
         <!-- <mesh filename="package://my_robot/description/drive_wheel.obj" scale="1.0 1.0 1.0"/> -->

File: src/my_robot/description/robot.urdf.xacro (robot description, xacro)
@@ -13,24 +13,25 @@
   joint_name="left_wheel_joint"
   parent_link="base_link"
-  xyz_pos="0.078 0.22 -0.2"/>
+  xyz_pos="-0.076 0.22 -0.2"
+  wheel_flipping="0"/>
+  <!-- <xacro:drive_wheel -->
   <xacro:drive_wheel
   wheel_name="right_wheel_link"
   joint_name="right_wheel_joint"
   parent_link="base_link"
-  xyz_pos="0.078 -0.22 -0.2"/>
+  xyz_pos="-0.076 -0.22 -0.2"
+  wheel_flipping="3.1415"/>
   <!-- <xacro:castor_wheel/> -->
   <xacro:castor_wheel
-  xyz_pos="-0.2 0 -0.225"/>
+  xyz_pos="0.2 0 -0.228"/>
   <!-- <xacro:robot_cover/> -->
   <xacro:robot_cover
-  xyz_pos="-0.06 0.0 0.05"/>s
-  <!-- define a root base_link -->
-  <link name="map"/>
-  <!-- fixed joint to attach chassis -->
+  xyz_pos="0.06 0.0 0.05"/>
+    <!-- <link name="map"/>
   <joint name="base_to_chassis" type="fixed">
     <parent link="map"/>
     <child link="base_link"/>
     <origin xyz="0 0 0" rpy="0 0 0"/>
-  </joint>
+  </joint> -->
 </xacro:macro>
 </robot>

Commit message: streamlining paths

File: src/my_robot/description/castor_wheel.urdf.xacro (robot description, xacro)
@@ -4,4 +4,5 @@
   <xacro:property name="parent_link" value="base_link"/>
   <xacro:property name="child_link"  value="castor_wheel"/>
+  <xacro:property name="mesh_path_castor_wheel" value="file://$(find my_robot)/mesh/castor_wheel.obj"/>
   <link name="castor_wheel">
     <inertial>
@@ -13,5 +14,6 @@
       <origin rpy="0 0 0" xyz="0 0 0"/>
       <geometry>
-        <mesh filename="file://$(find my_robot)/description/castor_wheel.obj" scale="1.0 1.0 1.0"/>
+        <!-- <mesh filename="file://$(find my_robot)/description/castor_wheel.obj" scale="1.0 1.0 1.0"/> -->
+        <mesh filename="${mesh_path_castor_wheel}"/>
       </geometry>
       <material name="white">
@@ -22,5 +24,6 @@
       <origin rpy="0 0 0" xyz="0 0 0"/>
       <geometry>
-        <mesh filename="file://$(find my_robot)/description/castor_wheel.obj" scale="1.0 1.0 1.0"/>
+        <mesh filename="${mesh_path_castor_wheel}"/>
+        <!-- <mesh filename="file://$(find my_robot)/description/castor_wheel.obj" scale="1.0 1.0 1.0"/> -->
         <!-- you could also specify the collision (for the castor_wheel) with a "box" tag: -->
         <!-- <box size=".06 .06 .06"/> -->

File: src/my_robot/description/chassis.urdf.xacro (robot description, xacro)
@@ -1,4 +1,5 @@
 <?xml version="1.0" ?>
 <robot xmlns:xacro="http://www.ros.org/wiki/xacro" name="chassis">
+  <xacro:property name="mesh_path_chassis" value="file://$(find my_robot)/mesh/chassis.obj"/>
   <xacro:macro name="chassis" params="">
     <link name="base_link">
@@ -12,5 +13,6 @@
         <geometry>
           <!-- <mesh filename="package://my_robot/description/chassis.obj" scale="1.0 1.0 1.0"/> -->
-          <mesh filename="file://$(find my_robot)/description/chassis.obj"/>
+          <!-- <mesh filename="file://$(find my_robot)/description/chassis.obj"/> -->
+          <mesh filename="${mesh_path_chassis}"/>
         </geometry>
         <material name="white">
@@ -22,5 +24,6 @@
         <geometry>
           <!-- <mesh filename="package://my_robot/description/chassis.obj" scale="1.0 1.0 1.0"/> -->
-          <mesh filename="file://$(find my_robot)/description/chassis.obj"/>
+          <!-- <mesh filename="file://$(find my_robot)/description/chassis.obj"/> -->
+          <mesh filename="${mesh_path_chassis}"/>
         </geometry>
       </collision>

File: src/my_robot/description/drive_wheel.urdf.xacro (robot description, xacro)
@@ -2,4 +2,5 @@
 <robot xmlns:xacro="http://www.ros.org/wiki/xacro" name="drive_wheel.urdf">
   <xacro:macro name="drive_wheel" params="wheel_name joint_name parent_link xyz_pos wheel_flipping">
+  <xacro:property name="mesh_path_drive_wheel" value="file://$(find my_robot)/mesh/drive_wheel.obj"/>
   <link name="${wheel_name}">
     <inertial>
@@ -12,5 +13,6 @@
       <geometry>
         <!-- <mesh filename="package://my_robot/description/drive_wheel.obj" scale="1.0 1.0 1.0"/> -->
-        <mesh filename="file://$(find my_robot)/description/drive_wheel.obj"/>
+        <!-- <mesh filename="file://$(find my_robot)/description/drive_wheel.obj"/> -->
+        <mesh filename="${mesh_path_drive_wheel}"/>
       </geometry>
       <material name="white">
@@ -22,5 +24,6 @@
       <geometry>
         <!-- <mesh filename="package://my_robot/description/drive_wheel.obj" scale="1.0 1.0 1.0"/> -->
-        <mesh filename="file://$(find my_robot)/description/drive_wheel.obj"/>
+        <!-- <mesh filename="file://$(find my_robot)/description/drive_wheel.obj"/> -->
+        <mesh filename="${mesh_path_drive_wheel}"/>
       </geometry>
     </collision>

File: src/my_robot/description/robot_cover.urdf.xacro (robot description, xacro)
@@ -1,4 +1,5 @@
 <?xml version="1.0" ?>
 <robot xmlns:xacro="http://www.ros.org/wiki/xacro" name="robot_cover.urdf">
+<xacro:property name="mesh_path_robot_cover" value="file://$(find my_robot)/mesh/robot_cover.obj"/>
 <xacro:macro name="robot_cover" params="xyz_pos">
   <link name="robot_cover">
@@ -11,5 +12,6 @@
       <origin rpy="0 0 0" xyz="0 0 0"/>
       <geometry>
-        <mesh filename="file://$(find my_robot)/description/robot_cover.obj" scale="1.0 1.0 1.0"/>
+        <mesh filename="${mesh_path_robot_cover}"/>
+        <!-- <mesh filename="file://$(find my_robot)/description/robot_cover.obj" scale="1.0 1.0 1.0"/> -->
       </geometry>
       <material name="white">
@@ -20,5 +22,6 @@
       <origin rpy="0 0 0" xyz="0 0 0"/>
       <geometry>
-        <mesh filename="file://$(find my_robot)/description/robot_cover.obj" scale="1.0 1.0 1.0"/>
+      <mesh filename="${mesh_path_robot_cover}"/>
+        <!-- <mesh filename="file://$(find my_robot)/description/robot_cover.obj" scale="1.0 1.0 1.0"/> -->
         <!-- you could also specify the collision (for the robot_cover) with a "box" tag: -->
         <!-- <box size=".06 .06 .06"/> -->
